Commit message: Add 4x Livox Mid-360 LiDARs and wide-angle camera to URDF
Replace single 2D base_laser with full sensor suite matching real X30:
- lidar_front_up:   front face, tilted up  → /x30/lidar_front_up/points
- lidar_front_down: front face, tilted down → /x30/lidar_front_down/points
- lidar_rear_up:    rear face,  tilted up  → /x30/lidar_rear_up/points
- lidar_rear_down:  rear face,  tilted down → /x30/lidar_rear_down/points
- camera_front: 90 deg FOV, 640x480 @ 30Hz → /x30/camera/image_raw

2D scan slice from front-up LiDAR retained on /x30/scan for AMCL/move_base.
Each 3D sensor: 360 deg horizontal, 32-beam vertical, 30m range, 10Hz.

File: src/x30_urdf/X30/urdf/X30.urdf (robot description, URDF)
Before this commit: robot X30, 19 links, 18 joints
Links:
- removed link base_laser
- added link camera_front, mass 0.05; visual box size=0.03 0.06 0.03
- added link lidar_front_down, mass 0.07; visual cylinder length=0.04 radius=0.025
- added link lidar_front_up, mass 0.07; visual cylinder length=0.04 radius=0.025
- added link lidar_rear_down, mass 0.07; visual cylinder length=0.04 radius=0.025
- added link lidar_rear_up, mass 0.07; visual cylinder length=0.04 radius=0.025
Joints:
- removed joint base_to_laser
- added joint base_to_camera_front: type fixed, parent base_link, child camera_front, origin xyz=0.22 0 0.13 rpy=0 0.15 0
- added joint base_to_lidar_front_down: type fixed, parent base_link, child lidar_front_down, origin xyz=0.22 0 0.01 rpy=0 0.5 0
- added joint base_to_lidar_front_up: type fixed, parent base_link, child lidar_front_up, origin xyz=0.22 0 0.10 rpy=0 -0.3 0
- added joint base_to_lidar_rear_down: type fixed, parent base_link, child lidar_rear_down, origin xyz=-0.22 0 0.01 rpy=0 0.5 3.14159
- added joint base_to_lidar_rear_up: type fixed, parent base_link, child lidar_rear_up, origin xyz=-0.22 0 0.10 rpy=0 -0.3 3.14159
